Commit message: bugs related to Gazebo 7.x fixed, found in: https://answers.ros.org/question/236122/diffdrive-odometry-source-is-missing/ https://github.com/ros-simulation/gazebo_ros_pkgs/issues/488 https://afsyaw.wordpress.com/2017/01/12/running-the-pioneer-3dx-in-gazebo-and-ros-kinetic/

File: p3dx_description/urdf/pioneer3dx.xacro (robot description, xacro)
@@ -92,5 +92,5 @@
 			<origin xyz="0 0 0" rpy="0 0 0" />
 			<geometry>
-				<box size="0 0 0" />
+				<box size="0.01 0.01 0.01" />
 			</geometry>
 		</collision>
@@ -125,5 +125,5 @@
 			<origin xyz="0 0 0" rpy="0 0 0" />
 			<geometry>
-				<box size="0 0 0" />
+				<box size="0.01 0.01 0.01" />
 			</geometry>
 		</collision>
@@ -188,5 +188,5 @@
 			<origin rpy="0 0 0" xyz="0 0 0" />
 			<geometry>
-				<box size="0 0 0" />
+				<box size="0.01 0.01 0.01" />
 			</geometry>
 		</collision>

File: p3dx_description/urdf/pioneer3dx_wheel.xacro (robot description, xacro)
@@ -71,5 +71,5 @@
 				<origin xyz="0 0 0" rpy="0 0 0" />
 				<geometry>
-					<box size="0 0 0" />
+					<box size="0.01 0.01 0.01" />
 				</geometry>
 			</collision>
